File: Unit1-04/Unit1-04.kicad_pcb (KiCad board)
At the start: 2 copper layers, 16 parts, among them Q1 BC547, Q2 BC547, Q3 BC547, Q4 BC547, Q5 BC547, SW1 SW_SPDT, SW2 SW_SPDT

Commit message: Added comment on PCB
Other:
- board text added: "Created By Cristiano S November 8th 2023 XNOR Gate with Transistors"
